Commit message: can convert xacro to urdf

File: akira_description/urdf/akira.urdf (robot description, URDF)
Before this commit: robot akira, 21 links, 20 joints
Links:
- removed link face_link
- removed link right_arm_base_link
- removed link right_arm_elbow_flex_link
- removed link right_arm_forearm_flex_link
- removed link right_arm_shoulder_lift_L_link
- removed link right_arm_shoulder_lift_R_link
- removed link right_arm_shoulder_pan_link
- removed link right_arm_shoulder_roll_link
- removed link right_arm_wrist_flex_link
- removed link right_gripper_link
Joints:
- removed joint right_arm_base_joint
- removed joint right_arm_elbow_flex_joint
- removed joint right_arm_forearm_flex_joint
- removed joint right_arm_shoulder_lift_L_joint
- removed joint right_arm_shoulder_lift_R_joint
- removed joint right_arm_shoulder_pan_joint
- removed joint right_arm_shoulder_roll_joint
- removed joint right_arm_wrist_flex_joint
- removed joint right_gripper_joint
- removed joint torso_face_joint
