Commit message: 2017/10/24

File: akira_description/urdf/akira.xacro (robot description, xacro)
@@ -10,10 +10,4 @@
    <property name="arm_offset_y" value="-0.20" />
    <property name="arm_offset_z" value="0.20" />
-   -->
-   <!-- face_offset_z= ${torso_size_z}/2 + ${face_size_z}/2 -->
-   <!--
-   <property name="face_offset_x" value="-0.03" />
-   <property name="face_offset_y" value="0.0" />
-   <property name="face_offset_z" value="0.532" />
    -->
    <property name="camera_offset_x" value="0.1" />
@@ -54,10 +48,4 @@
    </gripper>
    -->
-   <!-- Attach the face -->
-   <!--
-   <face name="face" parent="torso" color="Danboru">
-     <origin xyz="${face_offset_x} ${face_offset_y} ${face_offset_z}" rpy="0 0 0" />
-   </face>
-   -->
    <!-- Attach the camera -->
    <camera name="camera" parent="torso" color="Black">

Commit message: 2017/10/25

File: akira_description/urdf/akira.xacro (robot description, xacro)
@@ -2,19 +2,19 @@
 <robot name="akira" xmlns:xacro="http://ros.org/wiki/xacro">
    <!-- Define a number of dimensions using properties -->
-   <property name="PI" value="3.14159"/>
-   <property name="torso_offset_x" value="0.0" />
-   <property name="torso_offset_y" value="0.0" />
-   <property name="torso_offset_z" value="0.55" />
+   <xacro:property name="PI" value="3.14159"/>
+   <xacro:property name="torso_offset_x" value="0.0" />
+   <xacro:property name="torso_offset_y" value="0.0" />
+   <xacro:property name="torso_offset_z" value="0.55" />
    <!--
-   <property name="arm_offset_x" value="0.1" />
-   <property name="arm_offset_y" value="-0.20" />
-   <property name="arm_offset_z" value="0.20" />
+   <xacro:property name="arm_offset_x" value="0.1" />
+   <xacro:property name="arm_offset_y" value="-0.20" />
+   <xacro:property name="arm_offset_z" value="0.20" />
    -->
-   <property name="camera_offset_x" value="0.1" />
-   <property name="camera_offset_y" value="0.0" />
-   <property name="camera_offset_z" value="0.695" />
-   <property name="laser_offset_x" value="0.19" />
-   <property name="laser_offset_y" value="0.0" />
-   <property name="laser_offset_z" value="0.16" />
+   <xacro:property name="camera_offset_x" value="0.1" />
+   <xacro:property name="camera_offset_y" value="0.0" />
+   <xacro:property name="camera_offset_z" value="0.695" />
+   <xacro:property name="laser_offset_x" value="0.19" />
+   <xacro:property name="laser_offset_y" value="0.0" />
+   <xacro:property name="laser_offset_z" value="0.16" />
    <!-- Include all component files -->
    <xacro:include filename="$(find akira_description)/urdf/materials.urdf.xacro" />

Commit message: attach camera on the robot

File: akira_description/urdf/akira.xacro (robot description, xacro)
@@ -13,5 +13,5 @@
    <xacro:property name="camera_offset_x" value="0.1" />
    <xacro:property name="camera_offset_y" value="0.0" />
-   <xacro:property name="camera_offset_z" value="0.695" />
+   <xacro:property name="camera_offset_z" value="0.420" />
    <xacro:property name="laser_offset_x" value="0.19" />
    <xacro:property name="laser_offset_y" value="0.0" />

Commit message: maybe complete prototype

File: akira_description/urdf/akira.xacro (robot description, xacro)
@@ -30,8 +30,9 @@
    <xacro:include filename="$(find akira_description)/urdf/kinect.urdf.xacro" />
    <xacro:include filename="$(find akira_description)/urdf/laser.urdf.xacro" />
+   <xacro:include filename="$(find akira_description)/urdf/akira.gazebo" />
    <!-- Add the base and wheels -->
    <base name="base" color="Black"/>
    <!-- Attach the torso -->
-   <torso name="torso" parent="base" color="Danboru">
+   <torso name="torso" parent="base" color="Orange">
       <origin xyz="${torso_offset_x} ${torso_offset_y} ${torso_offset_z}" rpy="0 0 0" />
    </torso>
@@ -53,5 +54,5 @@
    </camera>
    <!-- Attach the laser -->
-   <laser parent="base" color="DarkGrey">
+   <laser parent="base" color="Grey">
       <origin xyz="${laser_offset_x} ${laser_offset_y} ${laser_offset_z}" rpy="0 0 0 " />
    </laser>

File: akira_description/urdf/akira_arm.urdf.xacro (robot description, xacro)
@@ -2,5 +2,5 @@
 <robot name="arm" xmlns:xacro="http://ros.org/wiki/xacro">
   <xacro:include filename="$(find akira_description)/urdf/arm_hardware.xacro" />
-  <macro name="arm" params="side reflect parent color *origin">
+  <xacro:macro name="arm" params="side reflect parent color *origin">
     <link name="${side}_arm_base_link" />
     <joint name="${side}_arm_base_joint" type="fixed">
@@ -51,4 +51,4 @@
       <axis xyz="0 0 1" />
     </RS405CB_revolute>
-  </macro>
+  </xacro:macro>
 </robot>

File: akira_description/urdf/akira_base_with_laser.xacro (robot description, xacro)
@@ -2,7 +2,7 @@
 <robot name="akira" xmlns:xacro="http://ros.org/wiki/xacro">
    <!-- Define a number of dimensions using properties -->
-   <property name="laser_offset_x" value="0.19" />
-   <property name="laser_offset_y" value="0.0" />
-   <property name="laser_offset_z" value="0.16" />
+   <xacro:property name="laser_offset_x" value="0.19" />
+   <xacro:property name="laser_offset_y" value="0.0" />
+   <xacro:property name="laser_offset_z" value="0.16" />
    <!-- Include all component files -->
    <xacro:include filename="$(find akira_description)/urdf/materials.urdf.xacro" />

File: akira_description/urdf/akira_face.urdf.xacro (robot description, xacro)
@@ -2,10 +2,10 @@
 <robot name="face" xmlns:xacro="http://ros.org/wiki/xacro">
  <!-- FACE_DEPTH: doesn't include its back horn-->
-  <property name="face_size_x" value="0.300" />
-  <property name="face_size_y" value="0.438" />
-  <property name="face_size_z" value="0.294" />
-  <property name="FACE_MESH_SCALE" value="1.0" />
+  <xacro:property name="face_size_x" value="0.300" />
+  <xacro:property name="face_size_y" value="0.438" />
+  <xacro:property name="face_size_z" value="0.294" />
+  <xacro:property name="FACE_MESH_SCALE" value="1.0" />
   <!-- Define the face -->
-  <macro name="face" params="parent name color *origin">
+  <xacro:macro name="face" params="parent name color *origin">
     <joint name="${parent}_${name}_joint" type="fixed">
       <xacro:insert_block name="origin" />
@@ -29,4 +29,4 @@
       </collision>
       </link>
-    </macro>
+    </xacro:macro>
 </robot>

File: akira_description/urdf/akira_gripper.urdf.xacro (robot description, xacro)
@@ -1,6 +1,6 @@
 <?xml version="1.0"?>
 <robot name="gripper" xmlns:xacro="http://ros.org/wiki/xacro">
-  <property name="PI" value="3.14159"/>
-  <macro name="gripper" params="side reflect parent color *origin">
+  <xacro:property name="PI" value="3.14159"/>
+  <xacro:macro name="gripper" params="side reflect parent color *origin">
     <!-- gripper base joint -->
     <!--RS405CB_revolute parent="${parent}" name="${side}_gripper_base" vlimit="1.571" llimit="0" ulimit="1.57">
@@ -53,4 +53,4 @@
     </link>
 -->
-   </macro>
+   </xacro:macro>
 </robot>

File: akira_description/urdf/akira_torso.urdf.xacro (robot description, xacro)
@@ -2,10 +2,10 @@
 <robot name="torso" xmlns:xacro="http://ros.org/wiki/xacro">
   <!-- Define a number of dimensions using properties -->
-  <property name="torso_size_x" value="0.29" />
-  <property name="torso_size_y" value="0.46" />
-  <property name="torso_size_z" value="0.77" />
-  <property name="TORSO_MESH_SCALE" value="1.0" />
+  <xacro:property name="torso_size_x" value="0.29" />
+  <xacro:property name="torso_size_y" value="0.46" />
+  <xacro:property name="torso_size_z" value="0.77" />
+  <xacro:property name="TORSO_MESH_SCALE" value="1.0" />
   <!-- Define the torso -->
-  <macro name="torso" params="parent name color *origin">
+  <xacro:macro name="torso" params="parent name color *origin">
     <joint name="${parent}_${name}_joint" type="fixed">
       <xacro:insert_block name="origin" />
@@ -31,4 +31,4 @@
       </collision>
       </link>
-    </macro>
+    </xacro:macro>
 </robot>

File: akira_description/urdf/akira_vehicle.urdf.xacro (robot description, xacro)
@@ -2,19 +2,19 @@
 <robot name="base" xmlns:xacro="http://ros.org/wiki/xacro">
 	<!-- Define a number of dimensions using properties -->
-	<property name="base_radius" value="0.25" />
-	<property name="base_length" value="0.3" />
-	<property name="wheel_radius" value="0.15" />
-	<property name="wheel_length" value="0.1" />
-	<property name="wheel_axis_length" value="0.25" />
-	<property name="wheel_offset_x" value="0" />
-	<property name="wheel_offset_y" value="0" />
-	<property name="wheel_offset_z" value="0" />
-	<property name="PI" value="3.1415" />
-	<property name="SIN30" value="0.5" />
-	<property name="COS30" value="0.8660" />
-	<property name="base_mesh_scale" value="1.0" />
+	<xacro:property name="base_radius" value="0.25" />
+	<xacro:property name="base_length" value="0.3" />
+	<xacro:property name="wheel_radius" value="0.15" />
+	<xacro:property name="wheel_length" value="0.1" />
+	<xacro:property name="wheel_axis_length" value="0.25" />
+	<xacro:property name="wheel_offset_x" value="0" />
+	<xacro:property name="wheel_offset_y" value="0" />
+	<xacro:property name="wheel_offset_z" value="0" />
+	<xacro:property name="PI" value="3.1415" />
+	<xacro:property name="SIN30" value="0.5" />
+	<xacro:property name="COS30" value="0.8660" />
+	<xacro:property name="base_mesh_scale" value="1.0" />
 	<!-- define a wheel -->
 	<!-- Link & joint -->
-	<macro name="wheel" params="suffix parent reflect color">
+	<xacro:macro name="wheel" params="suffix parent reflect color">
 	  <!-- joint -->
 	  <joint name="${parent}_${suffix}_wheel_joint" type="fixed">
@@ -36,8 +36,8 @@
 	    </visual>
 	  </link>
-	</macro>
+	</xacro:macro>
 	<!--  -->
 	<!-- The base link -->
-	<macro name="base" params="name color">
+	<xacro:macro name="base" params="name color">
 	  <!-- link -->
 	  <link name="${name}_link">
@@ -57,5 +57,5 @@
 	    </collision>
 	  </link>
-	</macro>
+	</xacro:macro>
 	<!-- The role of the base_footprint is essentially to define
 	     the elevation of the base above the ground. -->

File: akira_description/urdf/akira_with_arm.xacro (robot description, xacro)
@@ -2,11 +2,11 @@
 <robot name="akira" xmlns:xacro="http://ros.org/wiki/xacro">
    <!-- Define a number of dimensions using properties -->
-   <property name="PI" value="3.14159"/>
-   <property name="torso_offset_x" value="0.0" />
-   <property name="torso_offset_y" value="0.0" />
-   <property name="torso_offset_z" value="0.55" />
-   <property name="arm_offset_x" value="0.1" />
-   <property name="arm_offset_y" value="-0.20" />
-   <property name="arm_offset_z" value="0.20" />
+   <xacro:property name="PI" value="3.14159"/>
+   <xacro:property name="torso_offset_x" value="0.0" />
+   <xacro:property name="torso_offset_y" value="0.0" />
+   <xacro:property name="torso_offset_z" value="0.55" />
+   <xacro:property name="arm_offset_x" value="0.1" />
+   <xacro:property name="arm_offset_y" value="-0.20" />
+   <xacro:property name="arm_offset_z" value="0.20" />
    <!-- Include all component files -->
    <xacro:include filename="$(find akira_description)/urdf/materials.urdf.xacro" />

File: akira_description/urdf/akira_with_face.xacro (robot description, xacro)
@@ -2,11 +2,11 @@
 <robot name="akira" xmlns:xacro="http://ros.org/wiki/xacro">
   <!-- Define a number of dimensions using properties -->
-  <property name="torso_offset_x" value="0.0" />
-  <property name="torso_offset_y" value="0.0" />
-  <property name="torso_offset_z" value="0.55" />
+  <xacro:property name="torso_offset_x" value="0.0" />
+  <xacro:property name="torso_offset_y" value="0.0" />
+  <xacro:property name="torso_offset_z" value="0.55" />
   <!-- face_offset_z= ${torso_size_z}/2 + ${face_size_z}/2 -->
-  <property name="face_offset_x" value="0.0" />
-  <property name="face_offset_y" value="0.0" />
-  <property name="face_offset_z" value="0.532" />
+  <xacro:property name="face_offset_x" value="0.0" />
+  <xacro:property name="face_offset_y" value="0.0" />
+  <xacro:property name="face_offset_z" value="0.532" />
   <!-- Include all component files -->
   <xacro:include filename="$(find akira_description)/urdf/materials.urdf.xacro" />

File: akira_description/urdf/akira_with_kinect.xacro (robot description, xacro)
@@ -2,10 +2,10 @@
 <robot name="akira" xmlns:xacro="http://ros.org/wiki/xacro">
   <!-- Define a number of dimensions using properties -->
-  <property name="torso_offset_x" value="0.0" />
-  <property name="torso_offset_y" value="0.0" />
-  <property name="torso_offset_z" value="0.55" />
-  <property name="camera_offset_x" value="0.1" />
-  <property name="camera_offset_y" value="0.0" />
-  <property name="camera_offset_z" value="0.665" />
+  <xacro:property name="torso_offset_x" value="0.0" />
+  <xacro:property name="torso_offset_y" value="0.0" />
+  <xacro:property name="torso_offset_z" value="0.55" />
+  <xacro:property name="camera_offset_x" value="0.1" />
+  <xacro:property name="camera_offset_y" value="0.0" />
+  <xacro:property name="camera_offset_z" value="0.665" />
   <!-- include all component files -->
   <xacro:include filename="$(find akira_description)/urdf/materials.urdf.xacro" />

File: akira_description/urdf/akira_with_torso.xacro (robot description, xacro)
@@ -2,7 +2,7 @@
 <robot name="akira" xmlns:xacro="http://ros.org/wiki/xacro">
   <!-- Define a number of dimensions using properties -->
-  <property name="torso_offset_x" value="0.0" />
-  <property name="torso_offset_y" value="0.0" />
-  <property name="torso_offset_z" value="0.55" />
+  <xacro:property name="torso_offset_x" value="0.0" />
+  <xacro:property name="torso_offset_y" value="0.0" />
+  <xacro:property name="torso_offset_z" value="0.55" />
   <!-- Include all component files -->
   <xacro:include filename="$(find akira_description)/urdf/materials.urdf.xacro" />

File: akira_description/urdf/arm_hardware.xacro (robot description, xacro)
@@ -2,30 +2,30 @@
 <robot name="arm_hardware" xmlns:xacro="http://ros.org/wiki/xacro">
   <!-- RS405CB_DEPTH: doesn't include its back horn-->
-  <property name="RS405CB_WIDTH" value="0.033" />
-  <property name="RS405CB_HEIGHT" value="0.043" />
-  <property name="RS405CB_DEPTH" value="0.045" />
-  <property name="VH_6_W" value="0.03" />
-  <property name="VH_6_H" value="0.045" />
-  <property name="VH_6_D" value="0.054" />
-  <property name="VH_5_W" value="0.032" />
-  <property name="VH_5_H" value="0.032" />
-  <property name="VH_5_D" value="0.047" />
-  <property name="VH_4_W" value="0.032" />
-  <property name="VH_4_H" value="0.032" />
-  <property name="VH_4_D" value="0.047" />
-  <property name="VH_3_W" value="0.022" />
-  <property name="VH_3_H" value="0.037" />
-  <property name="VH_3_D" value="0.055" />
-  <property name="VH_2_W" value="0.032" />
-  <property name="VH_2_H" value="0.032" />
-  <property name="VH_2_D" value="0.047" />
-  <property name="VH_1A_W" value="0.022" />
-  <property name="VH_1A_H" value="0.037" />
-  <property name="VH_1A_D" value="0.055" />
-  <property name="VH_1B_W" value="0.032" />
-  <property name="VH_1B_H" value="0.032" />
-  <property name="VH_1B_D" value="0.047" />
-  <property name="PI" value="3.14159" />
-  <property name="RS405CB_MESH_SCALE" value="0.001" />
+  <xacro:property name="RS405CB_WIDTH" value="0.033" />
+  <xacro:property name="RS405CB_HEIGHT" value="0.043" />
+  <xacro:property name="RS405CB_DEPTH" value="0.045" />
+  <xacro:property name="VH_6_W" value="0.03" />
+  <xacro:property name="VH_6_H" value="0.045" />
+  <xacro:property name="VH_6_D" value="0.054" />
+  <xacro:property name="VH_5_W" value="0.032" />
+  <xacro:property name="VH_5_H" value="0.032" />
+  <xacro:property name="VH_5_D" value="0.047" />
+  <xacro:property name="VH_4_W" value="0.032" />
+  <xacro:property name="VH_4_H" value="0.032" />
+  <xacro:property name="VH_4_D" value="0.047" />
+  <xacro:property name="VH_3_W" value="0.022" />
+  <xacro:property name="VH_3_H" value="0.037" />
+  <xacro:property name="VH_3_D" value="0.055" />
+  <xacro:property name="VH_2_W" value="0.032" />
+  <xacro:property name="VH_2_H" value="0.032" />
+  <xacro:property name="VH_2_D" value="0.047" />
+  <xacro:property name="VH_1A_W" value="0.022" />
+  <xacro:property name="VH_1A_H" value="0.037" />
+  <xacro:property name="VH_1A_D" value="0.055" />
+  <xacro:property name="VH_1B_W" value="0.032" />
+  <xacro:property name="VH_1B_H" value="0.032" />
+  <xacro:property name="VH_1B_D" value="0.047" />
+  <xacro:property name="PI" value="3.14159" />
+  <xacro:property name="RS405CB_MESH_SCALE" value="0.001" />
   <!--macro name="RS405CB_fixed" params="parent name *origin">
     <joint name="${name}_joint" type="fixed">
@@ -56,6 +56,6 @@
       </collision>
     </link>
-  </macro-->
-  <macro name="RS405CB_revolute" params="parent name llimit ulimit vlimit *origin *axis">
+  </xacro:macro-->
+  <xacro:macro name="RS405CB_revolute" params="parent name llimit ulimit vlimit *origin *axis">
     <joint name="${name}_joint" type="revolute">
       <xacro:insert_block name="origin" />
@@ -89,6 +89,6 @@
       </collision>
     </link>
-  </macro>
-  <macro name="finger" params="parent name color *origin">
+  </xacro:macro>
+  <xacro:macro name="finger" params="parent name color *origin">
     <joint name="${name}_joint" type="fixed">
       <xacro:insert_block name="origin" />
@@ -118,4 +118,4 @@
       </collision>
     </link>
-  </macro>
+  </xacro:macro>
 </robot>

File: akira_description/urdf/kinect.urdf.xacro (robot description, xacro)
@@ -2,11 +2,11 @@
 <robot name="kinect" xmlns:xacro="http://ros.org/wiki/xacro">
    <!-- Define a number of dimensions using properties -->
-   <property name="kinect_size_x" value="0.07271" />
-   <property name="kinect_size_y" value="0.27794" />
-   <property name="kinect_size_z" value="0.070" />
-   <property name="camera_mesh_scale" value="1.0" />
-   <property name="PI" value="3.1415" />
+   <xacro:property name="kinect_size_x" value="0.07271" />
+   <xacro:property name="kinect_size_y" value="0.27794" />
+   <xacro:property name="kinect_size_z" value="0.070" />
+   <xacro:property name="camera_mesh_scale" value="1.0" />
+   <xacro:property name="PI" value="3.1415" />
    <!-- Define a camera link for a Kinect -->
-   <macro name="camera" params="parent name color *origin">
+   <xacro:macro name="camera" params="parent name color *origin">
       <joint name="${parent}_${name}_joint" type="fixed">
          <xacro:insert_block name="origin" />
@@ -115,4 +115,4 @@
       </joint>
       -->
-   </macro>
+   </xacro:macro>
 </robot>

File: akira_description/urdf/laser.urdf.xacro (robot description, xacro)
@@ -3,5 +3,5 @@
   <!-- A box-and-cylinder model of the Hokuyo URG-04LX-UG01 laser scanner -->
   <!-- Define the laser macro -->
-  <macro name="laser" params="parent color *origin">
+  <xacro:macro name="laser" params="parent color *origin">
     <joint name="${parent}_laser_bottom_joint" type="fixed">
       <xacro:insert_block name="origin" />
@@ -64,7 +64,5 @@
           <cylinder length="0.0175" radius=".0185"/>
         </geometry>
-        <material name="red">
-           <color rgba="0.8 0.1 0.1 1.0"/>
-        </material>
+        <material name="Red" />
      </visual>
      <collision>
@@ -86,4 +84,4 @@
      <origin xyz="0 0 0.0145" rpy="0 0 0" />
    </joint>
-  </macro>
+  </xacro:macro>
  </robot>
